File: design/pcb/ventmon_t0.4.sch (EAGLE design)
At the start: 77 parts, among them IC1 BME280BM280-HAT, J6 Header-16, J7 Header-12, U1 W5500, U2 ADS1115IDGST, Y1 25MHz

Commit message: Moved pressure sensors to accomodate small tube
Parts:
- removed X2: (no value), con-molex:KK-156-4
- added J4: (no value), SparkFun-Connectors:CONN_04POLAR
Connections:
- net +3V3: now also J4.2; no longer X2-2.S
- net BTNA: now also J4.4; no longer X2-4.S
- net BTNB: now also J4.3; no longer X2-3.S
- net GND: now also J4.1; no longer X2-1.S
Changed lines of the file:
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@@
 <part name="+3V6" library="supply1" deviceset="+3V3" device="" value="+3V3D"/>
 <part name="U$3" library="microbuilder" deviceset="GND" device=""/>
-<part name="X2" library="con-molex" library_urn="urn:adsk.eagle:library:165" deviceset="KK-156-4" device="" package3d_urn="urn:adsk.eagle:package:8078802/1"/>
 <part name="R16" library="microbuilder" deviceset="RESISTOR" device="0805" value="10K"/>
 <part name="+3V22" library="supply1" deviceset="+3V3" device="" value="+3V3D"/>
@@
 <part name="R18" library="microbuilder" deviceset="RESISTOR" device="0805" value="10K"/>
 <part name="U$12" library="microbuilder" deviceset="GND" device=""/>
+<part name="J4" library="SparkFun-Connectors" library_urn="urn:adsk.eagle:library:513" deviceset="CONN_04" device="POLAR" package3d_urn="urn:adsk.eagle:package:38087/1"/>
 </parts>
 <sheets>
@@
 <attribute name="VALUE" x="-9.144" y="-87.63" size="1.27" layer="96"/>
 </instance>
-<instance part="X2" gate="-1" x="-58.42" y="-10.16" smashed="yes" rot="R180">
-<attribute name="NAME" x="-60.96" y="-9.398" size="1.524" layer="95" rot="R180"/>
-<attribute name="VALUE" x="-57.658" y="-11.557" size="1.778" layer="96" rot="R180"/>
-</instance>
-<instance part="X2" gate="-2" x="-58.42" y="-7.62" smashed="yes" rot="R180">
-<attribute name="NAME" x="-60.96" y="-6.858" size="1.524" layer="95" rot="R180"/>
-</instance>
-<instance part="X2" gate="-3" x="-58.42" y="-5.08" smashed="yes" rot="R180">
-<attribute name="NAME" x="-60.96" y="-4.318" size="1.524" layer="95" rot="R180"/>
-</instance>
-<instance part="X2" gate="-4" x="-58.42" y="-2.54" smashed="yes" rot="R180">
-<attribute name="NAME" x="-60.96" y="-1.778" size="1.524" layer="95" rot="R180"/>
-</instance>
 <instance part="R16" gate="G$1" x="-34.29" y="-15.24" smashed="yes" rot="R90">
 <attribute name="NAME" x="-36.322" y="-17.78" size="1.27" layer="95" font="vector" rot="R90"/>
@@
 <instance part="U$12" gate="G$1" x="-27.94" y="-24.13" smashed="yes">
 <attribute name="VALUE" x="-29.464" y="-26.67" size="1.27" layer="96"/>
+</instance>
+<instance part="J4" gate="G$1" x="-63.5" y="-7.62" smashed="yes">
+<attribute name="VALUE" x="-68.58" y="-14.986" size="1.778" layer="96" font="vector"/>
+<attribute name="NAME" x="-68.58" y="0.508" size="1.778" layer="95" font="vector"/>
 </instance>
 </instances>
@@
 </segment>
 <segment>
-<pinref part="X2" gate="-1" pin="S"/>
-<wire x1="-55.88" y1="-10.16" x2="-50.8" y2="-10.16" width="0.1524" layer="91"/>
+<wire x1="-58.42" y1="-10.16" x2="-50.8" y2="-10.16" width="0.1524" layer="91"/>
 <pinref part="U$4" gate="G$1" pin="GND"/>
 <wire x1="-50.8" y1="-10.16" x2="-50.8" y2="-13.97" width="0.1524" layer="91"/>
+<pinref part="J4" gate="G$1" pin="1"/>
 </segment>
 <segment>
@@
 </segment>
 <segment>
-<pinref part="X2" gate="-2" pin="S"/>
-<wire x1="-55.88" y1="-7.62" x2="-48.26" y2="-7.62" width="0.1524" layer="91"/>
+<wire x1="-58.42" y1="-7.62" x2="-48.26" y2="-7.62" width="0.1524" layer="91"/>
 <wire x1="-48.26" y1="-7.62" x2="-48.26" y2="-12.7" width="0.1524" layer="91"/>
 <pinref part="+3V22" gate="G$1" pin="+3V3"/>
 <wire x1="-48.26" y1="-12.7" x2="-40.64" y2="-12.7" width="0.1524" layer="91"/>
+<pinref part="J4" gate="G$1" pin="2"/>
 </segment>
 </net>
@@
 </segment>
 <segment>
-<pinref part="X2" gate="-3" pin="S"/>
 <pinref part="R16" gate="G$1" pin="2"/>
-<wire x1="-55.88" y1="-5.08" x2="-34.29" y2="-5.08" width="0.1524" layer="91"/>
+<wire x1="-58.42" y1="-5.08" x2="-34.29" y2="-5.08" width="0.1524" layer="91"/>
 <wire x1="-34.29" y1="-5.08" x2="-34.29" y2="-10.16" width="0.1524" layer="91"/>
 <wire x1="-34.29" y1="-5.08" x2="-30.48" y2="-5.08" width="0.1524" layer="91"/>
 <label x="-33.02" y="-5.08" size="1.778" layer="95"/>
+<pinref part="J4" gate="G$1" pin="3"/>
 </segment>
 </net>
@@
 </segment>
 <segment>
-<pinref part="X2" gate="-4" pin="S"/>
 <pinref part="R18" gate="G$1" pin="2"/>
 <wire x1="-26.67" y1="-10.16" x2="-26.67" y2="-2.54" width="0.1524" layer="91"/>
-<wire x1="-26.67" y1="-2.54" x2="-55.88" y2="-2.54" width="0.1524" layer="91"/>
+<wire x1="-26.67" y1="-2.54" x2="-58.42" y2="-2.54" width="0.1524" layer="91"/>
 <wire x1="-26.67" y1="-2.54" x2="-22.86" y2="-2.54" width="0.1524" layer="91"/>
 <label x="-25.4" y="-2.54" size="1.778" layer="95"/>
-</segment>
-</net>
+<pinref part="J4" gate="G$1" pin="4"/>
+</segment>
+</net>
